File: hardware/boards/glasgow-revB0/glasgow.sch (KiCad schematic (older format))
At the start: 77 parts, among them J1 USB_B_Micro, J4 Conn_01x02, U1 CY7C68013A-56LTX, U15 TPD3S014, U2 CAT24M01W, U3 CAT24C256W, U4 ICE40UP5K-SG48ITR, U7 LM3880MF-1AF, U8 MIC5355-S4YMME, Y1 24M

Commit message: Updated revB0 to KiCad V5 and bumped revision from B to B0.
Also added bit more information to the board layout sheet legend.
Parts:
- MK1, MK2, MK3, MK4: symbol Mechanical:Mounting_Hole_PAD -> glasgow-rescue:Mounting_Hole_PAD-Mechanical
- MK5, MK6: symbol Mechanical:Mounting_Hole -> glasgow-rescue:Mounting_Hole-Mechanical
- TP1, TP2, TP3, TP4, TP5, TP6, TP7: symbol Connector:Test_Point -> glasgow-rescue:Test_Point-Connector
- U4: symbol FPGA_Lattice:ICE40UP5K-SG48ITR -> glasgow-rescue:ICE40UP5K-SG48ITR-FPGA_Lattice
Changed lines of the file:
@@
 Title "Base Board"
 Date ""
-Rev "B"
+Rev "B0"
 Comp "whitequark research"
 Comment1 "Glasgow Debug Tool"
@@
 NoConn ~ 1100 4350
 $Comp
-L Mechanical:Mounting_Hole_PAD MK1
+L glasgow-rescue:Mounting_Hole_PAD-Mechanical MK1
 U 1 1 5AD602A3
 P 900 7050
@@
 $EndComp
 $Comp
-L Mechanical:Mounting_Hole_PAD MK2
+L glasgow-rescue:Mounting_Hole_PAD-Mechanical MK2
 U 1 1 5AD64D62
 P 1100 7050
@@
 $EndComp
 $Comp
-L Mechanical:Mounting_Hole_PAD MK3
+L glasgow-rescue:Mounting_Hole_PAD-Mechanical MK3
 U 1 1 5AD64DAE
 P 1300 7050
@@
 $EndComp
 $Comp
-L Mechanical:Mounting_Hole_PAD MK4
+L glasgow-rescue:Mounting_Hole_PAD-Mechanical MK4
 U 1 1 5AD64E04
 P 1500 7050
@@
 CLKIF
 $Comp
-L FPGA_Lattice:ICE40UP5K-SG48ITR U4
+L glasgow-rescue:ICE40UP5K-SG48ITR-FPGA_Lattice U4
 U 1 1 5ADBCDAC
 P 7250 3100
@@
 $EndComp
 $Comp
-L FPGA_Lattice:ICE40UP5K-SG48ITR U4
+L glasgow-rescue:ICE40UP5K-SG48ITR-FPGA_Lattice U4
 U 2 1 5ADBCF53
 P 5700 2950
@@
 $EndComp
 $Comp
-L FPGA_Lattice:ICE40UP5K-SG48ITR U4
+L glasgow-rescue:ICE40UP5K-SG48ITR-FPGA_Lattice U4
 U 3 1 5ADBD03F
 P 5800 4900
@@
 $EndComp
 $Comp
-L FPGA_Lattice:ICE40UP5K-SG48ITR U4
+L glasgow-rescue:ICE40UP5K-SG48ITR-FPGA_Lattice U4
 U 4 1 5ADD0B90
 P 8350 1350
@@
 	4850 4150 4900 4150
 $Comp
-L Connector:Test_Point TP1
+L glasgow-rescue:Test_Point-Connector TP1
 U 1 1 5ADB3D1E
 P 900 2700
@@
 $EndComp
 $Comp
-L Connector:Test_Point TP2
+L glasgow-rescue:Test_Point-Connector TP2
 U 1 1 5AE0012C
 P 10450 5700
@@
 $EndComp
 $Comp
-L Connector:Test_Point TP3
+L glasgow-rescue:Test_Point-Connector TP3
 U 1 1 5AE0058E
 P 10850 5700
@@
 	7900 950  8250 950
 $Comp
-L Mechanical:Mounting_Hole MK5
+L glasgow-rescue:Mounting_Hole-Mechanical MK5
 U 1 1 5ADBCE07
 P 1750 7000
@@
 $EndComp
 $Comp
-L Mechanical:Mounting_Hole MK6
+L glasgow-rescue:Mounting_Hole-Mechanical MK6
 U 1 1 5ADBD505
 P 1950 7000
@@
 NoConn ~ 8600 3050
 $Comp
-L Connector:Test_Point TP4
+L glasgow-rescue:Test_Point-Connector TP4
 U 1 1 5AE223CE
 P 2200 5150
@@
 $EndComp
 $Comp
-L Connector:Test_Point TP5
+L glasgow-rescue:Test_Point-Connector TP5
 U 1 1 5AE22A82
 P 2300 5150
@@
 	2300 5150 2300 5050
 $Comp
-L Connector:Test_Point TP6
+L glasgow-rescue:Test_Point-Connector TP6
 U 1 1 5AE93638
 P 4950 5700
@@
 $EndComp
 $Comp
-L Connector:Test_Point TP7
+L glasgow-rescue:Test_Point-Connector TP7
 U 1 1 5B12B6CA
 P 4950 5800
