File: hardware/boards/glasgow/io_banks.sch (KiCad schematic (older format))
At the start: 16 parts, among them J10 Conn_01x03, J4 Conn_01x02, J5 Conn_02x22_Odd_Even, U30 ICE40HX8K-BG121

Commit message: Added 1BitSquared BOM keys to the schematic.
Parts:
- C33: Key (none) -> cap-cer-0402-100n
- D10, D6: Key (none) -> led-0603-blu
- D7, D9: Key (none) -> led-0603-pnk
- D8: Key (none) -> led-0603-wht
- J10: Key (none) -> conn-th-005in-3-1-hdr
- J4: Key (none) -> conn-th-01in-2-1-hdr-ra
- J5: Key (none) -> conn-smd-005in-22-2-hdr
- R10: Key (none) -> res-0402-130
- R11, R20, R21: Key (none) -> res-0402-2k2
- R22: Key (none) -> res-0402-390
- R23: Key (none) -> res-0402-604
- U30: Key (none) -> ic-ice40hx8k-bg121
Changed lines of the file:
@@
 F 2 "Package_BGA:BGA-121_9.0x9.0mm_Layout11x11_P0.8mm_Ball0.4mm_Pad0.35mm_NSMD" H 4750 3000 50  0001 C CNN
 F 3 "http://www.latticesemi.com/Products/FPGAandCPLD/iCE40" H 3900 5450 50  0001 C CNN
+F 4 "ic-ice40hx8k-bg121" H 0   0   50  0001 C CNN "Key"
 	2    4750 4450
 	-1   0    0    -1
@@
 F 2 "Package_BGA:BGA-121_9.0x9.0mm_Layout11x11_P0.8mm_Ball0.4mm_Pad0.35mm_NSMD" H 8250 2750 50  0001 C CNN
 F 3 "http://www.latticesemi.com/Products/FPGAandCPLD/iCE40" H 7400 5200 50  0001 C CNN
+F 4 "ic-ice40hx8k-bg121" H 0   0   50  0001 C CNN "Key"
 	4    8250 4200
 	-1   0    0    -1
@@
 F 2 "Connector_PinHeader_1.27mm:PinHeader_2x22_P1.27mm_Vertical_SMD" H 10000 4300 50  0001 C CNN
 F 3 "~" H 10000 4300 50  0001 C CNN
+F 4 "conn-smd-005in-22-2-hdr" H 0   0   50  0001 C CNN "Key"
 	1    10000 4300
 	1    0    0    -1
@@
 F 4 "Wurth Electronics" H -450 150 50  0001 C CNN "Mfg"
 F 5 "150060GS75000" H -450 150 50  0001 C CNN "MPN"
+F 6 "led-0603-blu" H 0   0   50  0001 C CNN "Key"
 	1    9800 1050
 	-1   0    0    1
@@
 F 4 "Wurth Electronics" H -450 150 50  0001 C CNN "Mfg"
 F 5 "150060GS75000" H -450 150 50  0001 C CNN "MPN"
+F 6 "led-0603-pnk" H 0   0   50  0001 C CNN "Key"
 	1    9800 1250
 	-1   0    0    1
@@
 F 4 "Wurth Electronics" H -450 150 50  0001 C CNN "Mfg"
 F 5 "150060GS75000" H -450 150 50  0001 C CNN "MPN"
+F 6 "led-0603-wht" H 0   0   50  0001 C CNN "Key"
 	1    9800 1450
 	-1   0    0    1
@@
 F 4 "Wurth Electronics" H -450 150 50  0001 C CNN "Mfg"
 F 5 "150060YS75000" H -450 150 50  0001 C CNN "MPN"
+F 6 "led-0603-pnk" H 0   0   50  0001 C CNN "Key"
 	1    9800 1650
 	-1   0    0    1
@@
 F 4 "Wurth Electronics" H -450 150 50  0001 C CNN "Mfg"
 F 5 "150060RS75000" H -450 150 50  0001 C CNN "MPN"
+F 6 "led-0603-blu" H 0   0   50  0001 C CNN "Key"
 	1    9800 1850
 	-1   0    0    1
@@
 F 4 "Yageo" H -450 150 50  0001 C CNN "Mfg"
 F 5 "RC0603FR-132K2L" H -450 150 50  0001 C CNN "MPN"
+F 6 "res-0402-2k2" H 0   0   50  0001 C CNN "Key"
 	1    9450 1050
 	0    -1   1    0
@@
 F 4 "Yageo" H -450 150 50  0001 C CNN "Mfg"
 F 5 "RC0603FR-13390RL" H -450 150 50  0001 C CNN "MPN"
+F 6 "res-0402-390" H 0   0   50  0001 C CNN "Key"
 	1    9450 1650
 	0    -1   1    0
@@
 F 4 "Yageo" H -450 150 50  0001 C CNN "Mfg"
 F 5 "RC0603FR-07604RL" H -450 150 50  0001 C CNN "MPN"
+F 6 "res-0402-604" H 0   0   50  0001 C CNN "Key"
 	1    9450 1850
 	0    -1   1    0
@@
 F 4 "Yageo" H -450 150 50  0001 C CNN "Mfg"
 F 5 "RC0603FR-132K2L" H -450 150 50  0001 C CNN "MPN"
+F 6 "res-0402-2k2" H 0   0   50  0001 C CNN "Key"
 	1    9450 1250
 	0    -1   1    0
@@
 F 4 "Yageo" H -450 150 50  0001 C CNN "Mfg"
 F 5 "RC0603FR-132K2L" H -450 150 50  0001 C CNN "MPN"
+F 6 "res-0402-2k2" H 0   0   50  0001 C CNN "Key"
 	1    9450 1450
 	0    -1   1    0
@@
 F 4 "Taiyo Yuden" H 2200 1250 50  0001 C CNN "Mfg"
 F 5 "TMK107BJ154KA-T" H 2200 1250 50  0001 C CNN "MPN"
+F 6 "cap-cer-0402-100n" H 0   0   50  0001 C CNN "Key"
 	1    8850 2650
 	1    0    0    -1
@@
 F 2 "Connector_PinHeader_1.27mm:PinHeader_1x03_P1.27mm_Vertical" H 2350 3550 50  0001 C CNN
 F 3 "~" H 2350 3550 50  0001 C CNN
+F 4 "conn-th-005in-3-1-hdr" H 0   0   50  0001 C CNN "Key"
 	1    2350 3550
 	1    0    0    -1
@@
 F 4 "Molex" H -8000 100 50  0001 C CNN "Mfg"
 F 5 "22-05-3021" H -8000 100 50  0001 C CNN "MPN"
+F 6 "conn-th-01in-2-1-hdr-ra" H 0   0   50  0001 C CNN "Key"
 	1    2600 2950
 	1    0    0    1
@@
 F 4 "Yageo" H -8000 100 50  0001 C CNN "Mfg"
 F 5 "AC0603FR-07130RL" H -8000 100 50  0001 C CNN "MPN"
+F 6 "res-0402-130" H 0   0   50  0001 C CNN "Key"
 	1    2350 2650
 	1    0    0    1
@@
 F 2 "Package_BGA:BGA-121_9.0x9.0mm_Layout11x11_P0.8mm_Ball0.4mm_Pad0.35mm_NSMD" H 1300 2800 50  0001 C CNN
 F 3 "http://www.latticesemi.com/Products/FPGAandCPLD/iCE40" H 450 5250 50  0001 C CNN
+F 4 "ic-ice40hx8k-bg121" H 0   0   50  0001 C CNN "Key"
 	1    1300 4250
 	-1   0    0    -1
