File: hardware/boards/glasgow/io_buffer.sch (KiCad schematic (older format))
At the start: 52 parts, among them J2 Conn_02x10_Odd_Even, J6 Conn_01x08, J7 Conn_01x08, U10 DAC081C081CIMK, U11 TPS73101DBV, U16 SN74LVC1T45DRL, U17 SN74LVC1T45DRL, U18 SN74LVC1T45DRL, U19 SN74LVC1T45DRL, U19 TCA9534, U20 SN74LVC1T45DRL, U21 SN74LVC1T45DRL, U33 TCA9517, U5 SN74LVC1T45DRL, U6 SN74LVC1T45DRL, U9 ADC081C021CIMM

Commit message: Added 1BitSquared BOM keys to the schematic.
Parts:
- C30, C32, C35, C36, C38, C39, C40, C47, C48, C49, C50, C51, C52, C53, C54, C55, C56, C57, C58, C59, C86, C87: Key (none) -> cap-cer-0402-100n
- C37: Key (none) -> cap-cer-0401-12n
- C82, C83: Key (none) -> cap-cer-0603-4u7
- J2: Key (none) -> conn-th-01in-10-1-hdr-shr
- J6, J7: Key (none) -> conn-th-005in-8-1-hdr
- R20, R21, R38, R39: Key (none) -> res-0402-10k
- R22: Key (none) -> res-0402-49k9
- R23: Key (none) -> res-0402-59k
- R24: Key (none) -> res-0402-24k3
- RN1, RN2: value R_Pack08 -> 100; Key (none) -> res-0602cv-array-8-100
- RN6: Key (none) -> res-0602cv-array-8-10k
- U10: Key (none) -> ic-sot23-6-dac081c081cimK
- U11: Key (none) -> ic-sot23-5-tps73101dbv
- U16, U17, U18, U19, U20, U21, U5, U6: Key (none) -> ic-sot563-sn74lvc1t45drl
- U19: Key (none) -> ic-tssop16-tca9534
- U33: Key (none) -> ic-vssop8-tca9517
- U9: Key (none) -> ic-msop8-adc081c021cimm
